Commit message: feat(data_collected.py): 新增随机动作采样器和数据收集 fix(panda_pushing_env.py): 更新物体参数并添加中间物体 fix(sim_env_vis.py): 调整动作采样和循环次数

File: assets/objects/disk/disk_big.urdf (robot description, URDF)
Before this commit: robot disk, 1 links, 0 joints
Links:
- link baseLink: geometry collision cylinder length=0.04 radius=0.08; visual cylinder length=0.04 radius=0.08
